File: pcb/minicoralbridge.kicad_pcb (KiCad board)
At the start: 4 copper layers, 34 x 47 mm, 7 parts, among them J1 MOLEX 679100002, J2 Bus_PCI_Express_x1

Commit message: more changes
Parts:
- removed R1: 0, Resistor_SMD:R_0603_1608Metric
- added REF**: OSHW-Logo2_9.8x8mm_SilkScreen, Symbol:OSHW-Logo2_9.8x8mm_SilkScreen, F.Cu at (82.3, 82.0)
- J1: value MOLEX 679100002 -> MOLEX 0679101002 / TE 1775862
Connections:
- J1 pad 11: /MINI_REFCLK_N -> /MINI_REFCLK_P
- J1 pad 13: /MINI_REFCLK_P -> /MINI_REFCLK_N
- J1 pad 2: /+3V3FUSED -> +3V3
- J1 pad 24: /+3V3FUSED -> +3V3
- J1 pad 39: /+3V3FUSED -> +3V3
- J1 pad 41: /+3V3FUSED -> +3V3
- J1 pad 52: /+3V3FUSED -> +3V3
Routing:
- net +3V3: track 19.4 -> 71.3 mm, vias 1 -> 7
- net /+3V3FUSED: track 51.4 -> 0.00 mm, vias 6 -> 0
- net Net-(J2-~{PRSNT2}): track 33.9 -> 22.3 mm, vias 1 -> 3
- net /CLKREQ: track 21.4 -> 27.0 mm
- net /MINI_REFCLK_P: track 23.1 -> 18.1 mm
- net GND: track 75.3 -> 71.6 mm, vias 38 -> 33
- net /MINI_PET0_P: track 21.0 -> 18.9 mm, vias 2 -> 0
- net /MINI_PET0_N: track 21.0 -> 18.9 mm, vias 2 -> 0
- net /MINI_PER0_P: track 16.0 -> 16.8 mm
- net /MINI_PER0_N: track 16.0 -> 16.8 mm
- net /MINI_REFCLK_N: track 18.7 -> 18.1 mm

Commit message: updates
Parts:
- removed the REF** at (94.5, 75.7)
- removed the REF** at (70.3, 75.7)
- added H1: SMSI-M2_H4mm_9774040243, Mounting_Wuerth:Mounting_Wuerth_WA-SMSI-M2_H4mm_9774040243, F.Cu at (70.3, 75.7)
- added H2: SMSI-M2_H4mm_9774040243, Mounting_Wuerth:Mounting_Wuerth_WA-SMSI-M2_H4mm_9774040243, F.Cu at (94.5, 75.7)
- J1: value MOLEX 0679101002 / TE 1775862 -> MOLEX 0679101002 / TE 2041119-1 (4mm)
Routing:
- net +3V3: track 71.3 -> 40.1 mm, vias 7 -> 5
- net GND: track 71.6 -> 68.1 mm, vias 33 -> 34
- net /CLKREQ: track 27.0 -> 26.4 mm
- added copper zone on B.Cu, net +3V3

Commit message: chchchchchanges
Parts:
- J1: value MOLEX 0679101002 / TE 2041119-1 (4mm) -> TE 2041262-1
Routing:
- net GND: track 68.1 -> 67.6 mm, vias 34 -> 37
- net /MINI_PER0_P: track 16.8 -> 17.4 mm
- net /MINI_PER0_N: track 16.8 -> 17.4 mm
- net unconnected-(J1-PadMP): vias 0 -> 8
