File: pcb/minicoralbridge.kicad_sch (KiCad schematic)
At the start: 4 parts, among them J1 MOLEX 679100002, J2 Bus_PCI_Express_x1

Commit message: more changes
Parts:
- removed R1: 0, Resistor_SMD:R_0603_1608Metric, symbol Device:R_Small
- J1: value MOLEX 679100002 -> MOLEX 0679101002 / TE 1775862
Connections:
- net +3V3FUSED is gone; now on net +3V3: J1.2 (+3V3AUX), J1.24 (+3V3AUX), J1.39 (+3V3AUX), J1.41 (+3V3AUX), J1.52 (+3V3AUX)
- net MINI_REFCLK_N: now also J1.13 (REFCLK+); no longer J1.11 (REFCLK-)
- net MINI_REFCLK_P: now also J1.11 (REFCLK-); no longer J1.13 (REFCLK+)
Other:
- moved on the sheet: J2, JP2

Commit message: updates
Parts:
- added H1, H2: SMSI-M2_H4mm_9774040243, Mounting_Wuerth:Mounting_Wuerth_WA-SMSI-M2_H4mm_9774040243, symbol Mechanical:MountingHole
- J1: value MOLEX 0679101002 / TE 1775862 -> TE 2041262-1
Other:
- note added: "Polarity reversal per PCIe spec"
- note removed: "LANE SWAP per PCIe spec"
Changed lines of the file:
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@@
+    (stroke (width 0) (type default))
+  )
+  (wire (pts (xy 58.42 50.8) (xy 60.96 50.8))
     (stroke (width 0) (type default))
   )
@@
     (stroke (width 0) (type default))
   )
+  (wire (pts (xy 102.87 78.74) (xy 110.49 78.74))
+    (stroke (width 0) (type default))
+  )
+  (wire (pts (xy 48.26 81.28) (xy 50.8 81.28))
+    (stroke (width 0) (type default))
+  )
   (wire (pts (xy 66.04 50.8) (xy 68.58 50.8))
     (stroke (width 0) (type default))
   )
-  (wire (pts (xy 102.87 78.74) (xy 110.49 78.74))
-    (stroke (width 0) (type default))
-  )
-  (wire (pts (xy 58.42 50.8) (xy 60.96 50.8))
-    (stroke (width 0) (type default))
-  )
-  (wire (pts (xy 48.26 81.28) (xy 50.8 81.28))
-    (stroke (width 0) (type default))
-  )
   (wire (pts (xy 48.26 109.22) (xy 50.8 109.22))
     (stroke (width 0) (type default))
@@
     (stroke (width 0) (type default))
   )
-  (text "LANE SWAP\nper PCIe spec" (at 21.59 81.28 0)
-    (effects (font (size 1.27 1.27)) (justify left bottom))
-  )
-  (text "LANE SWAP\nper PCIe spec" (at 21.59 74.93 0)
+  (rectangle (start 24.13 71.12) (end 49.53 90.17)
+    (stroke (width 0) (type default))
+    (fill (type color) (color 0 0 0 0.2))
+  )
+  (text "Polarity reversal\nper PCIe spec" (at 29.21 88.9 90)
     (effects (font (size 1.27 1.27)) (justify left bottom))
   )
@@
         (path "/7e71481c-d42b-4efe-a14b-0ecbd3e61cce"
           (reference "#PWR04") (unit 1)
+        )
+      )
+    )
+  )
+  (symbol (lib_id "Mechanical:MountingHole") (at 27.94 139.7 0) (unit 1)
+    (in_bom yes) (on_board yes) (dnp no) (fields_autoplaced)
+    (property "Reference" "H1" (at 30.48 139.065 0)
+      (effects (font (size 1.27 1.27)) (justify left))
+    )
+    (property "Value" "SMSI-M2_H4mm_9774040243" (at 30.48 141.605 0)
+      (effects (font (size 1.27 1.27)) (justify left))
+    )
+    (property "Footprint" "Mounting_Wuerth:Mounting_Wuerth_WA-SMSI-M2_H4mm_9774040243" (at 27.94 139.7 0)
+      (effects (font (size 1.27 1.27)) hide)
+    )
+    (property "Datasheet" "~" (at 27.94 139.7 0)
+      (effects (font (size 1.27 1.27)) hide)
+    )
+    (instances
+      (project "minicoralbridge"
+        (path "/7e71481c-d42b-4efe-a14b-0ecbd3e61cce"
+          (reference "H1") (unit 1)
+        )
+      )
+    )
+  )
+  (symbol (lib_id "Mechanical:MountingHole") (at 27.94 146.05 0) (unit 1)
+    (in_bom yes) (on_board yes) (dnp no) (fields_autoplaced)
+    (property "Reference" "H2" (at 30.48 145.415 0)
+      (effects (font (size 1.27 1.27)) (justify left))
+    )
+    (property "Value" "SMSI-M2_H4mm_9774040243" (at 30.48 147.955 0)
+      (effects (font (size 1.27 1.27)) (justify left))
+    )
+    (property "Footprint" "Mounting_Wuerth:Mounting_Wuerth_WA-SMSI-M2_H4mm_9774040243" (at 27.94 146.05 0)
+      (effects (font (size 1.27 1.27)) hide)
+    )
+    (property "Datasheet" "~" (at 27.94 146.05 0)
+      (effects (font (size 1.27 1.27)) hide)
+    )
+    (instances
+      (project "minicoralbridge"
+        (path "/7e71481c-d42b-4efe-a14b-0ecbd3e61cce"
+          (reference "H2") (unit 1)
         )
       )
@@
       (effects (font (size 1.27 1.27)) (justify left))
     )
-    (property "Value" "MOLEX 0679101002 / TE 1775862" (at 73.66 113.03 0)
-      (effects (font (size 1.27 1.27)) (justify left))
-    )
+    (property "Value" "TE 2041262-1" (at 73.66 113.03 0)
+      (effects (font (size 1.27 1.27)) (justify left))
+    )

Commit message: chchchchchanges
Other:
- note added: "alternate: 91304-68-052R2 (C404122)"
- note added: "alternate: TH162040CTJ (C3020128)"
Changed lines of the file:
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@@
     (fill (type color) (color 0 0 0 0.2))
+  )
+  (text "alternate: TH162040CTJ (C3020128)" (at 30.48 151.13 0)
+    (effects (font (size 1.27 1.27)) (justify left bottom))
   )
   (text "Polarity reversal\nper PCIe spec" (at 29.21 88.9 90)
     (effects (font (size 1.27 1.27)) (justify left bottom))
   )
+  (text "alternate: 91304-68-052R2 (C404122)" (at 73.66 116.84 0)
+    (effects (font (size 1.27 1.27)) (justify left bottom))
+  )
